File: basic-oscilloscope.sch (KiCad schematic (older format))
At the start: 30 parts, among them J1 9V_BATTERY, J2 12V_DC_JACK, U1 LT3032-3.3, U2 STM32F103C8Tx, Y1 Crystal, Y2 Crystal

Commit message: add hardware debounce
Parts:
- added C? (x5): 0.1u, symbol Device:CP
- added J?: CH1, symbol Connector:Conn_Coaxial
- added J?: CH2, symbol Connector:Conn_Coaxial
- added R? (x5): 1k, symbol Device:R
- added SW?: SW_SPST, symbol Switch:SW_SPST
- added SW? (x5): SW_Push, symbol Switch:SW_Push
- added U? (x5): 74HC14, symbol 74xx:74HC14
Connections:
- net 0: now also C?.2, C?.2, C?.2, C?.2, C?.2, SW?.1, SW?.1, SW?.1, SW?.1, SW?.1
- net at C1.1, C2.1, C3.1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: now also SW?.1 (A); no longer U1.14 (INP)
- new net: SW?.2 (B), U1.14 (INP)
- new net: C?.1, R?.1, U?.1 (x5)
- new net: R?.2, SW?.2 (x5)
- new net +: U?.2
- new net -: U?.2
- new net ACT_BUF: U?.2
- new net GND: J?.2 (Ext), J?.2 (Ext)
- new net HOLD_RUN: U?.2
- new net SEL_OK: U?.2
- new net TO_BUF: J?.1 (In)
- new net TO_BUF2: J?.1 (In)
Other:
- note added: "CONNECTORS\n"
- note added: "CONTROL\n"
- note added: "DO: Activate pull-ups for GPIO in code"
- moved on the sheet: C5, C6, U1A
