File: screen.sch (KiCad schematic (older format))
At the start: 1 part

Commit message: create TFT screen definition and instance
Other:
- note added: "SCREEN"
Changed lines of the file:
@@
 	0    -1   -1   0
 $EndComp
+Text Notes 5500 2100 0    168  ~ 34
+SCREEN
 $EndSCHEMATC
